File: contents.sch (KiCad schematic (older format))
At the start: 64 parts

Commit message: component values
Parts:
- removed D? (x2): D_ALT, symbol D_ALT
- removed Q? (x2): 2N2222, TO_SOT_Packages_THT:TO-92_Molded_Narrow, symbol BC237
- added D? (x5): 1N5819, symbol D_Schottky
- added Q? (x2): NTR4503NT1G, TO_SOT_Packages_SMD:SOT-23_Handsoldering, symbol Q_NMOS_GSD
- added R?: 1k, Resistors_ThroughHole:Resistor_Horizontal_RM10mm, symbol R
- added SP?: SPEAKER, symbol SPEAKER
- D? (x3): value LED -> KPT-1608SGC; footprint LEDs:LED-3MM -> LEDs:LED_0805_HandSoldering
- Q?: value 2N2222 -> NTR4503NT1G; footprint TO_SOT_Packages_THT:TO-92_Molded_Narrow -> TO_SOT_Packages_SMD:SOT-23_Handsoldering; symbol BC237 -> Q_NMOS_GSD
- Q?: footprint TO_SOT_Packages_THT:TO-92_Molded_Narrow -> TO_SOT_Packages_SMD:SOT-23_Handsoldering
- R? (x3): value 670 -> 1k
- R? (x3): value 220 -> 820
Connections:
- net +3V3: now also D?.1 (K)
- net +5V: now also R?.2, SP?.1
- net +VDC: now also D?.1 (K), D?.1 (K), D?.1 (K)
- net 1Wire: now also D?.1 (K), D?.2 (A)
- net BUZ: now also R?.2
- net GND: now also Q?.2 (E), Q?.2 (S), D?.2 (A), Q?.2 (S), Q?.2 (S); no longer Q?.3 (E)
- net at R?.1: now also Q?.1 (G) (x2)
- net at D?.1 (K), P?.2 (P2): now also D?.2 (A), Q?.3 (D) (x2)
- net at R?.1: now also Q?.1 (G); no longer Q?.2 (B)
- net at D?.1 (K), P?.2 (P2): now also Q?.3 (D), D?.2 (A); no longer Q?.1 (C)
- net at R?.1: now also Q?.1 (B)
- net at Q?.3 (C): now also R?.1, SP?.2
Other:
- note added: "3 SSR/Relay outputs :\nDriving power : Vin, 1A each"
- note removed: "3 SSR/Relay outputs :\nDriving power : Vin, 600mA each"
- moved on the sheet: Q?, R?
Changed lines of the file:
@@
 P 3100 4200
 F 0 "R?" V 3180 4200 50  0000 C CNN
-F 1 "670" V 3100 4200 50  0000 C CNN
+F 1 "1k" V 3100 4200 50  0000 C CNN
 F 2 "Resistors_ThroughHole:Resistor_Horizontal_RM10mm" V 3030 4200 50  0001 C CNN
 F 3 "" H 3100 4200 50  0000 C CNN
 	1    3100 4200
 	0    1    1    0
-$EndComp
-$Comp
-L BC237 Q?
-U 1 1 595CD6DF
-P 3650 4200
-F 0 "Q?" H 3850 4275 50  0000 L CNN
-F 1 "2N2222" H 3850 4200 50  0000 L CNN
-F 2 "TO_SOT_Packages_THT:TO-92_Molded_Narrow" H 3950 4400 50  0000 L CIN
-F 3 "" H 3650 4200 50  0000 L CNN
-	1    3650 4200
-	1    0    0    -1
 $EndComp
 $Comp
@@
 AR Path="/595CC9DA/595CD6E2" Ref="D?"  Part="1"
 F 0 "D?" H 3750 3800 50  0000 C CNN
-F 1 "LED" H 3750 3600 50  0000 C CNN
-F 2 "LEDs:LED-3MM" H 3750 3700 50  0001 C CNN
+F 1 "KPT-1608SGC" H 3800 3600 50  0000 C CNN
+F 2 "LEDs:LED_0805_HandSoldering" H 3750 3700 50  0001 C CNN
 F 3 "" H 3750 3700 50  0000 C CNN
 	1    3750 3700
@@
 P 3750 3350
 F 0 "R?" V 3830 3350 50  0000 C CNN
-F 1 "220" V 3750 3350 50  0000 C CNN
+F 1 "820" V 3750 3350 50  0000 C CNN
 F 2 "Resistors_ThroughHole:Resistor_Horizontal_RM10mm" V 3680 3350 50  0001 C CNN
 F 3 "" H 3750 3350 50  0000 C CNN
@@
 P 5200 4200
 F 0 "R?" V 5280 4200 50  0000 C CNN
-F 1 "670" V 5200 4200 50  0000 C CNN
+F 1 "1k" V 5200 4200 50  0000 C CNN
 F 2 "Resistors_ThroughHole:Resistor_Horizontal_RM10mm" V 5130 4200 50  0001 C CNN
 F 3 "" H 5200 4200 50  0000 C CNN
 	1    5200 4200
 	0    1    1    0
-$EndComp
-$Comp
-L BC237 Q?
-U 1 1 59A73F67
-P 5750 4200
-F 0 "Q?" H 5950 4275 50  0000 L CNN
-F 1 "2N2222" H 5950 4200 50  0000 L CNN
-F 2 "TO_SOT_Packages_THT:TO-92_Molded_Narrow" H 5400 4000 50  0000 L CIN
-F 3 "" H 5750 4200 50  0000 L CNN
-	1    5750 4200
-	1    0    0    -1
 $EndComp
 $Comp
@@
 P 5850 3700
 F 0 "D?" H 5850 3800 50  0000 C CNN
-F 1 "LED" H 5850 3600 50  0000 C CNN
-F 2 "LEDs:LED-3MM" H 5850 3700 50  0001 C CNN
+F 1 "KPT-1608SGC" H 5900 3600 50  0000 C CNN
+F 2 "LEDs:LED_0805_HandSoldering" H 5850 3700 50  0001 C CNN
 F 3 "" H 5850 3700 50  0000 C CNN
 	1    5850 3700
@@
 P 5850 3350
 F 0 "R?" V 5930 3350 50  0000 C CNN
-F 1 "220" V 5850 3350 50  0000 C CNN
+F 1 "820" V 5850 3350 50  0000 C CNN
 F 2 "Resistors_ThroughHole:Resistor_Horizontal_RM10mm" V 5780 3350 50  0001 C CNN
 F 3 "" H 5850 3350 50  0000 C CNN
@@
 	1    0    0    -1
 $EndComp
-$Comp
-L D_ALT D?
-U 1 1 59A74A6F
-P 4100 3550
-F 0 "D?" H 4100 3650 50  0000 C CNN
-F 1 "D_ALT" H 4100 3450 50  0000 C CNN
-F 2 "" H 4100 3550 50  0001 C CNN
-F 3 "" H 4100 3550 50  0001 C CNN
-	1    4100 3550
-	0    1    1    0
-$EndComp
-$Comp
-L D_ALT D?
-U 1 1 59A74C89
-P 6200 3550
-F 0 "D?" H 6200 3650 50  0000 C CNN
-F 1 "D_ALT" H 6200 3450 50  0000 C CNN
-F 2 "" H 6200 3550 50  0001 C CNN
-F 3 "" H 6200 3550 50  0001 C CNN
-	1    6200 3550
-	0    1    1    0
-$EndComp
 Text GLabel 800  4200 0    60   Input ~ 0
 SSR1
@@
 P 1200 4200
 F 0 "R?" V 1280 4200 50  0000 C CNN
-F 1 "670" V 1200 4200 50  0000 C CNN
+F 1 "1k" V 1200 4200 50  0000 C CNN
 F 2 "Resistors_ThroughHole:Resistor_Horizontal_RM10mm" V 1130 4200 50  0001 C CNN
 F 3 "" H 1200 4200 50  0000 C CNN
@@
 $EndComp
 $Comp
-L BC237 Q?
+L Q_NMOS_GSD Q?
 U 1 1 59A7538D
 P 1750 4200
 F 0 "Q?" H 1950 4275 50  0000 L CNN
-F 1 "2N2222" H 1950 4200 50  0000 L CNN
-F 2 "TO_SOT_Packages_THT:TO-92_Molded_Narrow" H 1950 4400 50  0000 L CIN
+F 1 "NTR4503NT1G" H 1950 4200 50  0000 L CNN
+F 2 "TO_SOT_Packages_SMD:SOT-23_Handsoldering" H 1200 4400 50  0000 L CIN
 F 3 "" H 1750 4200 50  0000 L CNN
 	1    1750 4200
@@
 P 1850 3700
 F 0 "D?" H 1850 3800 50  0000 C CNN
-F 1 "LED" H 1850 3600 50  0000 C CNN
-F 2 "LEDs:LED-3MM" H 1850 3700 50  0001 C CNN
+F 1 "KPT-1608SGC" H 1900 3600 50  0000 C CNN
+F 2 "LEDs:LED_0805_HandSoldering" H 1850 3700 50  0001 C CNN
 F 3 "" H 1850 3700 50  0000 C CNN
 	1    1850 3700
@@
 P 1850 3350
 F 0 "R?" V 1930 3350 50  0000 C CNN
-F 1 "220" V 1850 3350 50  0000 C CNN
+F 1 "820" V 1850 3350 50  0000 C CNN
 F 2 "Resistors_ThroughHole:Resistor_Horizontal_RM10mm" V 1780 3350 50  0001 C CNN
 F 3 "" H 1850 3350 50  0000 C CNN
@@
 Linear LDO regulator 5V ->3.3V, 1A
 Text Notes 4200 4750 0    60   ~ 0
-3 SSR/Relay outputs :\nDriving power : Vin, 600mA each
+3 SSR/Relay outputs :\nDriving power : Vin, 1A each
 Text Notes 10000 3650 0    60   ~ 0
 Accessory port 1 :\n+3.3V, i2c
@@
 	850  7050 1400 7050
 Wire Wire Line
-	1250 7050 1250 7000
+	1250 7000 1250 7200
 Connection ~ 1250 7050
 Wire Wire Line
@@
 Wire Notes Line
 	500  7800 500  6350
-Text Notes 550  7700 0    60   ~ 0
+Text Notes 2100 7800 0    60   ~ 0
 OneWire Bus\nTo connect DS18b20,\nfor example
-Text GLabel 3850 5300 0    60   Input ~ 0
+Text GLabel 3900 6400 0    60   Input ~ 0
 BUZ
 $Comp
 L R R?
 U 1 1 59B9D8A6
-P 4250 5500
-F 0 "R?" V 4330 5500 50  0000 C CNN
-F 1 "670" V 4250 5500 50  0000 C CNN
-F 2 "Resistors_ThroughHole:Resistor_Horizontal_RM10mm" V 4180 5500 50  0001 C CNN
-F 3 "" H 4250 5500 50  0000 C CNN
-	1    4250 5500
+P 4150 6400
+F 0 "R?" V 4230 6400 50  0000 C CNN
+F 1 "670" V 4150 6400 50  0000 C CNN
+F 2 "Resistors_ThroughHole:Resistor_Horizontal_RM10mm" V 4080 6400 50  0001 C CNN
+F 3 "" H 4150 6400 50  0000 C CNN
+	1    4150 6400
 	0    1    1    0
 $EndComp
@@
 L BC817 Q?
 U 1 1 59B9D9BD
-P 4750 5500
-F 0 "Q?" H 4950 5575 50  0000 L CNN
-F 1 "BC817" H 4950 5500 50  0000 L CNN
-F 2 "TO_SOT_Packages_THT:TO-92_Molded_Narrow" H 5050 5700 50  0000 L CIN
-F 3 "" H 4750 5500 50  0000 L CNN
-	1    4750 5500
-	1    0    0    -1
-$EndComp
+P 4600 6400
+F 0 "Q?" H 4800 6475 50  0000 L CNN
+F 1 "BC817" H 4800 6400 50  0000 L CNN
+F 2 "TO_SOT_Packages_SMD:SOT-23_Handsoldering" H 4900 6600 50  0000 L CIN
+F 3 "" H 4600 6400 50  0000 L CNN
+	1    4600 6400
+	1    0    0    -1
+$EndComp
+$Comp
+L D_Schottky D?
+U 1 1 59B9AD54
+P 4100 3550
+F 0 "D?" H 4100 3650 50  0000 C CNN
+F 1 "1N5819" H 4100 3450 50  0000 C CNN
+F 2 "" H 4100 3550 50  0001 C CNN
+F 3 "" H 4100 3550 50  0001 C CNN
+	1    4100 3550
+	0    1    1    0
+$EndComp
+$Comp
+L D_Schottky D?
+U 1 1 59B9AE45
+P 6200 3550
+F 0 "D?" H 6200 3650 50  0000 C CNN
+F 1 "1N5819" H 6200 3450 50  0000 C CNN
+F 2 "" H 6200 3550 50  0001 C CNN
+F 3 "" H 6200 3550 50  0001 C CNN
+	1    6200 3550
+	0    1    1    0
+$EndComp
+$Comp
+L D_Schottky D?
+U 1 1 59B9B36D
+P 2200 3500
+F 0 "D?" H 2200 3600 50  0000 C CNN
+F 1 "1N5819" H 2200 3400 50  0000 C CNN
+F 2 "" H 2200 3500 50  0001 C CNN
+F 3 "" H 2200 3500 50  0001 C CNN
+	1    2200 3500
+	0    1    1    0
+$EndComp
+Wire Wire Line
+	2200 3350 2200 3200
+Connection ~ 2200 3200
+Wire Wire Line
+	2200 3650 2200 3950
+Connection ~ 2200 3950
+$Comp
+L Q_NMOS_GSD Q?
+U 1 1 59B9C1B5
+P 3650 4200
+F 0 "Q?" H 3850 4275 50  0000 L CNN
+F 1 "NTR4503NT1G" H 3850 4200 50  0000 L CNN
+F 2 "TO_SOT_Packages_SMD:SOT-23_Handsoldering" H 3100 4400 50  0000 L CIN
+F 3 "" H 3650 4200 50  0000 L CNN
+	1    3650 4200
+	1    0    0    -1
+$EndComp
+$Comp
+L Q_NMOS_GSD Q?
+U 1 1 59B9C291
+P 5750 4200
+F 0 "Q?" H 5950 4275 50  0000 L CNN
+F 1 "NTR4503NT1G" H 5950 4200 50  0000 L CNN
+F 2 "TO_SOT_Packages_SMD:SOT-23_Handsoldering" H 5200 4400 50  0000 L CIN
+F 3 "" H 5750 4200 50  0000 L CNN
+	1    5750 4200
+	1    0    0    -1
+$EndComp
+$Comp
+L GND #PWR?
+U 1 1 59B9E716
+P 1250 7650
+F 0 "#PWR?" H 1250 7400 50  0001 C CNN
+F 1 "GND" H 1250 7500 50  0000 C CNN
+F 2 "" H 1250 7650 50  0000 C CNN
+F 3 "" H 1250 7650 50  0000 C CNN
+	1    1250 7650
+	1    0    0    -1
+$EndComp
+$Comp
+L D_Schottky D?
+U 1 1 59B9ECCE
+P 1250 7350
+F 0 "D?" H 1250 7450 50  0000 C CNN
+F 1 "1N5819" H 1250 7250 50  0000 C CNN
+F 2 "" H 1250 7350 50  0001 C CNN
+F 3 "" H 1250 7350 50  0001 C CNN
+	1    1250 7350
+	0    1    1    0
+$EndComp
+Wire Wire Line
+	1250 7500 1250 7650
+$Comp
+L D_Schottky D?
+U 1 1 59B9EFFE
+P 1050 6850
+F 0 "D?" H 1050 6950 50  0000 C CNN
+F 1 "1N5819" H 1050 6750 50  0000 C CNN
+F 2 "" H 1050 6850 50  0001 C CNN
+F 3 "" H 1050 6850 50  0001 C CNN
+	1    1050 6850
+	0    1    1    0
+$EndComp
+Wire Wire Line
+	1050 7050 1050 7000
+Connection ~ 1050 7050
+Wire Wire Line
+	1050 6700 1050 6650
+Wire Wire Line
+	1050 6650 1250 6650
+Connection ~ 1250 6650
+$Comp
+L SPEAKER SP?
+U 1 1 59B9FFA9
+P 5000 5800
+F 0 "SP?" H 4900 6050 50  0000 C CNN
+F 1 "SPEAKER" H 4900 5550 50  0000 C CNN
+F 2 "" H 5000 5800 50  0000 C CNN
+F 3 "" H 5000 5800 50  0000 C CNN
+	1    5000 5800
+	1    0    0    -1
+$EndComp
+Wire Wire Line
+	3900 6400 4000 6400
+Wire Wire Line
+	4300 6400 4400 6400
+$Comp
+L +5V #PWR?
+U 1 1 59BA44C8
+P 4700 5350
+F 0 "#PWR?" H 4700 5200 50  0001 C CNN
+F 1 "+5V" H 4700 5490 50  0000 C CNN
+F 2 "" H 4700 5350 50  0000 C CNN
+F 3 "" H 4700 5350 50  0000 C CNN
+	1    4700 5350
+	1    0    0    -1
+$EndComp
+Wire Wire Line
+	4700 5350 4700 5700
+Wire Wire Line
+	4700 5900 4700 6200
+$Comp
+L R R?
+U 1 1 59BA55B2
+P 4450 5800
+F 0 "R?" V 4530 5800 50  0000 C CNN
+F 1 "1k" V 4450 5800 50  0000 C CNN
+F 2 "Resistors_ThroughHole:Resistor_Horizontal_RM10mm" V 4380 5800 50  0001 C CNN
+F 3 "" H 4450 5800 50  0000 C CNN
+	1    4450 5800
+	-1   0    0    1
+$EndComp
+Wire Wire Line
+	4450 5650 4450 5550
+Wire Wire Line
+	4450 5550 4700 5550
+Connection ~ 4700 5550
+Wire Wire Line
+	4450 5950 4450 6050
+Wire Wire Line
+	4450 6050 4700 6050
+Connection ~ 4700 6050
+$Comp
+L GND #PWR?
+U 1 1 59BA5950
+P 4700 6850
+F 0 "#PWR?" H 4700 6600 50  0001 C CNN
+F 1 "GND" H 4700 6700 50  0000 C CNN
+F 2 "" H 4700 6850 50  0000 C CNN
+F 3 "" H 4700 6850 50  0000 C CNN
+	1    4700 6850
+	1    0    0    -1
+$EndComp
+Wire Wire Line
+	4700 6850 4700 6600
+$Comp
+L +5V #PWR?
+U 1 1 59BA606A
+P 6800 1250
+F 0 "#PWR?" H 6800 1100 50  0001 C CNN
+F 1 "+5V" H 6800 1390 50  0000 C CNN
+F 2 "" H 6800 1250 50  0000 C CNN
+F 3 "" H 6800 1250 50  0000 C CNN
+	1    6800 1250
+	1    0    0    -1
+$EndComp

Commit message: ADC values
Parts:
- added C12: 1u, Capacitors_ThroughHole:C_Rect_L7_W2.5_P5, symbol C
- gave numbers to parts that had none: 69
Connections:
- net P5V is gone; now on net +5V: C5.1, C6.1, C8.1, C9.1, L1.2, R19.1, U3.1 (VI)
- net +3V3: now also C12.1
- net +VDC: now also C1.1, C2.1, C3.1, D3.1 (K), R10.1, U1.3 (VIN); no longer D3.2 (A), P1.2 (P2), P2.2 (P2)
- net GND: now also C12.2
- new net: D3.2 (A), P1.2 (P2), P2.2 (P2)

Commit message: BOM
Parts:
- removed J1, J2, J4: Audio-Jack-3, symbol Audio-Jack-3
- added J4: Conn_01x06, Mylib:bornier6_2.54, symbol Conn_01x06
- C1, C8: footprint (none) -> Capacitors_SMD:CP_Elec_10x10.5
- C10, C12, C13, C14: footprint Capacitors_ThroughHole:C_Rect_L7_W2.5_P5 -> Capacitors_SMD:C_0805_HandSoldering
- C11: footprint (none) -> Capacitors_SMD:CP_Elec_6.3x7.7
- C2, C5, C6: footprint (none) -> Capacitors_SMD:C_1206_HandSoldering
- C3, C4, C7: footprint (none) -> Capacitors_SMD:C_0805_HandSoldering
- C9: footprint (none) -> Capacitors_SMD:CP_Elec_5x5.3
- D1, D10, D2, D5, D6, D8: footprint (none) -> Diodes_SMD:D_SOD-123
- D3: value D_Schottky -> DB2X41500L; footprint (none) -> Diodes_SMD:D_SOD-123
- J5: footprint (none) -> Connect:bornier2
- L1: value L_Core_Ferrite -> MSS7341-103MLD; footprint (none) -> Choke_SMD:Choke_SMD_7.3x7.3_H4.5
- P1: footprint Pin_Headers:Pin_Header_Straight_1x02 -> Connect:BARREL_JACK; symbol CONN_01X02 -> Barrel_Jack
- P2, P3, P4, P5: footprint Pin_Headers:Pin_Header_Straight_1x02 -> Connect:bornier2
- P6: footprint Pin_Headers:Pin_Header_Straight_1x04 -> Connect:Fan_Pin_Header_Straight_1x04
- P7: footprint Pin_Headers:Pin_Header_Straight_1x04 -> Connect:PINHEAD1-6
- Q3: footprint (none) -> TO_SOT_Packages_SMD:SOT-23_Handsoldering
- R10: renamed from R2; footprint Resistors_ThroughHole:Resistor_Horizontal_RM10mm -> Resistors_SMD:R_0805_HandSoldering
- R11: renamed from R3; footprint Resistors_ThroughHole:Resistor_Horizontal_RM10mm -> Resistors_SMD:R_0805_HandSoldering
- R12: renamed from R4; footprint Resistors_ThroughHole:Resistor_Horizontal_RM10mm -> Resistors_SMD:R_0805_HandSoldering
- R13: renamed from R5; footprint Resistors_ThroughHole:Resistor_Horizontal_RM10mm -> Resistors_SMD:R_0805_HandSoldering
- R14: renamed from R10; footprint (none) -> Resistors_SMD:R_0805_HandSoldering
- R15: renamed from R12; footprint (none) -> Resistors_SMD:R_0805_HandSoldering
- R16: renamed from R13; footprint Resistors_ThroughHole:Resistor_Horizontal_RM10mm -> Resistors_SMD:R_0805_HandSoldering
- R17: renamed from R14; footprint Resistors_ThroughHole:Resistor_Horizontal_RM10mm -> Resistors_SMD:R_0805_HandSoldering
- R18: renamed from R15; footprint Resistors_ThroughHole:Resistor_Horizontal_RM10mm -> Resistors_SMD:R_0805_HandSoldering
- R19: renamed from R16; footprint Resistors_ThroughHole:Resistor_Horizontal_RM10mm -> Resistors_SMD:R_0805_HandSoldering
- R20: renamed from R17; footprint Resistors_ThroughHole:Resistor_Horizontal_RM10mm -> Resistors_SMD:R_0805_HandSoldering
- R21: renamed from R18; footprint Resistors_ThroughHole:Resistor_Horizontal_RM10mm -> Resistors_SMD:R_0805_HandSoldering
- R22: renamed from R19; footprint (none) -> Resistors_SMD:R_0805_HandSoldering
- R23: renamed from R20; footprint (none) -> Resistors_SMD:R_0805_HandSoldering
- R24: renamed from R21; footprint (none) -> Resistors_SMD:R_0805_HandSoldering
- R25: renamed from R22; footprint Resistors_ThroughHole:Resistor_Horizontal_RM10mm -> Resistors_SMD:R_0805_HandSoldering
- R26: renamed from R25; footprint Resistors_ThroughHole:Resistor_Horizontal_RM10mm -> Resistors_SMD:R_0805_HandSoldering
- R27: renamed from R26; footprint Resistors_ThroughHole:Resistor_Horizontal_RM10mm -> Resistors_SMD:R_0805_HandSoldering
- R28: renamed from R27; footprint Resistors_ThroughHole:Resistor_Horizontal_RM10mm -> Resistors_SMD:R_0805_HandSoldering
- R29: renamed from R28; footprint Resistors_ThroughHole:Resistor_Horizontal_RM10mm -> Resistors_SMD:R_0805_HandSoldering
- R30, R31, R32: footprint Resistors_ThroughHole:Resistor_Horizontal_RM10mm -> Resistors_SMD:R_0805_HandSoldering
- R9: renamed from R1; footprint Resistors_ThroughHole:Resistor_Horizontal_RM10mm -> Resistors_SMD:R_0805_HandSoldering
- SP1: footprint (none) -> Capacitors_ThroughHole:CP_Radial_D16.0mm_P7.50mm
- U2: renamed from U1; footprint (none) -> TO_SOT_Packages_SMD:SOT-23-6_Handsoldering
- U3: footprint TO_SOT_Packages_THT:TO-220_Vertical -> TO_SOT_Packages_SMD:SOT-223-3Lead_TabPin2
- U4: footprint TO_SOT_Packages_SMD:SOT-23-5 -> TO_SOT_Packages_SMD:TSOT-23-5_HandSoldering
Connections:
- net +3V3: now also J4.1 (Pin_1), J4.4 (Pin_4)
- net 1Wire: now also J4.2 (Pin_2), J4.5 (Pin_5)
- net GND: now also P1.2, P1.3, J4.3 (Pin_3), J4.6 (Pin_6); no longer P1.1 (P1)
- net at D3.2 (A), P2.2 (P2): now also P1.1; no longer P1.2 (P2)
