File: contents.sch (KiCad schematic (older format))
At the start: 68 parts, among them J4 Conn_01x06, J5 Screw_Terminal_01x02, P1 Power jack, P2 Power, P3 SSR 1, P4 SSR 2, P5 SSR 3, P6 i2c_ext, P7 Ext, Q3 TSM2306, Q4 NTR4503NT1G, Q5 NTR4503NT1G, Q6 BC817, Q7 NTR4503NT1G, U2 TPS54302, U3 LM3940_SOT223, U4 LM321

Commit message: PCB created
Parts:
- J5: value Screw_Terminal_01x02 -> PWM
- RV1: footprint Potentiometers:Potentiometer_Bourns_3296W_3-8Zoll_Inline_ScrewUp -> Potentiometers:Potentiometer_Trimmer_Bourns_3266W
Changed lines of the file:
@@
 F 0 "RV1" H 9450 5100 50  0000 C CNN
 F 1 "1k" H 9450 5200 50  0000 C CNN
-F 2 "Potentiometers:Potentiometer_Bourns_3296W_3-8Zoll_Inline_ScrewUp" H 9450 5200 50  0001 C CNN
+F 2 "Potentiometers:Potentiometer_Trimmer_Bourns_3266W" H 9450 5200 50  0001 C CNN
 F 3 "" H 9450 5200 50  0000 C CNN
 	1    9450 5200
@@
 P 2700 5300
 F 0 "J5" H 2700 5400 50  0000 C CNN
-F 1 "Screw_Terminal_01x02" H 2900 5100 50  0000 C CNN
+F 1 "PWM" H 2900 5100 50  0000 C CNN
 F 2 "Connect:bornier2" H 2700 5300 50  0001 C CNN
 F 3 "" H 2700 5300 50  0001 C CNN

Commit message: Continued simplifiying
Parts:
- removed C1: 470uF, Capacitors_SMD:CP_Elec_10x10.5, symbol CP
- removed C2: 10uF, Capacitors_SMD:C_1206_HandSoldering, symbol C
- removed C3, C4: 100nF, Capacitors_SMD:C_0805_HandSoldering, symbol C
- removed C5, C6: 22uF, Capacitors_SMD:C_1206_HandSoldering, symbol C
- removed C7: 75pF, Capacitors_SMD:C_0805_HandSoldering, symbol C
- removed L1: MSS7341-103MLD, Choke_SMD:Choke_SMD_7.3x7.3_H4.5, symbol L_Core_Ferrite
- removed R14: 511k, Resistors_SMD:R_0805_HandSoldering, symbol R
- removed R15: 105k, Resistors_SMD:R_0805_HandSoldering, symbol R
- removed R22: 49.9, Resistors_SMD:R_0805_HandSoldering, symbol R
- removed R23: 100k, Resistors_SMD:R_0805_HandSoldering, symbol R
- removed R24: 13.3k, Resistors_SMD:R_0805_HandSoldering, symbol R
- removed U2: TPS54302, TO_SOT_Packages_SMD:SOT-23-6_Handsoldering, symbol TPS54302
- added U201: BuckModule, project_footprints:Buck-Module-1, symbol BuckModule
- J201: renamed from J4; footprint Mylib:bornier6_2.54 -> project_footprints:bornier6_2.54
- J202: renamed from J5; footprint Connect:bornier2 -> Connectors_Terminal_Blocks:TerminalBlock_bornier-2_P5.08mm
- P201: renamed from P1; footprint Connect:BARREL_JACK -> Connectors:BARREL_JACK
- P202: renamed from P2; footprint Connect:bornier2 -> Connectors_Terminal_Blocks:TerminalBlock_bornier-2_P5.08mm
- P203: renamed from P3; footprint Connect:bornier2 -> Connectors_Terminal_Blocks:TerminalBlock_bornier-2_P5.08mm
- P204: renamed from P4; footprint Connect:bornier2 -> Connectors_Terminal_Blocks:TerminalBlock_bornier-2_P5.08mm
- P205: renamed from P5; footprint Connect:bornier2 -> Connectors_Terminal_Blocks:TerminalBlock_bornier-2_P5.08mm
- P206: renamed from P6; footprint Connect:Fan_Pin_Header_Straight_1x04 -> Connectors:Fan_Pin_Header_Straight_1x04
- P207: renamed from P7; footprint Connect:PINHEAD1-6 -> Connectors:PINHEAD1-6
- SP201: renamed from SP1; footprint Capacitors_ThroughHole:CP_Radial_D16.0mm_P7.50mm -> Capacitors_THT:CP_Radial_D12.5mm_P7.50mm
- U202: renamed from U3; footprint TO_SOT_Packages_SMD:SOT-223-3Lead_TabPin2 -> TO_SOT_Packages_SMD:SOT-223-3_TabPin2
- renumbered C8 to C201, C9 to C202, C10 to C203, C11 to C204, C12 to C205, C13 to C206, C14 to C207, D1 to D201, D2 to D202, D3 to D203, D4 to D204, D5 to D205, D6 to D206, D7 to D207, D8 to D208, D9 to D209, D10 to D210, Q3 to Q201, Q4 to Q202, Q5 to Q203, Q6 to Q204, Q7 to Q205, R9 to R201, R10 to R202, R11 to R203, R12 to R204, R13 to R205, R16 to R206, R17 to R207, R18 to R208, R19 to R209, R20 to R210, R21 to R211, R25 to R212, R26 to R213, R27 to R214, R28 to R215, R29 to R216, R30 to R217, R31 to R218, R32 to R219, RV1 to RV201, U4 to U203
Connections:
- net +5V: now also U201.3 (OUT+)
- net +VDC: now also U201.1 (IN+)
- net GND: now also U201.2 (IN-), U201.4 (OUT-)
Other:
- note removed: "SMPS 9-28V -> 5V, 3A"
- moved on the sheet: C201
