File: Arpette.kicad_pcb (KiCad board)
At the start: 4 copper layers, 65 x 56 mm, 18 parts, among them J3 40HAT, J6 CONN_02X02, J9 CONN_01X02, Q1 DMG2305UX, Q2 DMMT5401, U2 CAT24C32

Commit message: PCB created
Parts:
- removed J6: CONN_02X02, Pin_Headers:Pin_Header_Straight_2x02
- removed J9: CONN_01X02, Pin_Headers:Pin_Header_Straight_1x02
- added C1: 470uF, Capacitors_SMD:CP_Elec_10x10.5, F.Cu at (221.7, 114.0)
- added C10: 1u, Capacitors_SMD:C_0805_HandSoldering, F.Cu at (236.0, 185.9)
- added C11: 470uF, low ESR, Capacitors_SMD:CP_Elec_6.3x7.7, F.Cu at (256.8, 172.1)
- added C12: 1u, Capacitors_SMD:C_0805_HandSoldering, F.Cu at (230.3, 193.4)
- added C13: 1u, Capacitors_SMD:C_0805_HandSoldering, F.Cu at (276.4, 164.2)
- added C14: 1u, Capacitors_SMD:C_0805_HandSoldering, F.Cu at (297.8, 160.0)
- added C15: 1n, Capacitors_SMD:C_0805_HandSoldering, F.Cu at (222.8, 164.4)
- added C16: 1n, Capacitors_SMD:C_0805_HandSoldering, F.Cu at (222.8, 160.8)
- added C17: 1n, Capacitors_SMD:C_0805_HandSoldering, F.Cu at (234.1, 165.6)
- added C18: 1n, Capacitors_SMD:C_0805_HandSoldering, F.Cu at (230.4, 186.0)
- added C19: 1n, Capacitors_SMD:C_0805_HandSoldering, F.Cu at (226.2, 154.5)
- added C2: 10uF, Capacitors_SMD:C_1206_HandSoldering, F.Cu at (214.7, 115.3)
- added C20: 1n, Capacitors_SMD:C_0805_HandSoldering, F.Cu at (232.2, 154.5)
- added C21: 1n, Capacitors_SMD:C_0805_HandSoldering, F.Cu at (243.8, 152.1)
- added C22: 1n, Capacitors_SMD:C_0805_HandSoldering, F.Cu at (248.8, 154.7)
- added C23: 47n, Capacitors_SMD:C_0805_HandSoldering, F.Cu at (228.6, 165.4)
- added C24: 470n, Capacitors_SMD:C_0805_HandSoldering, F.Cu at (216.1, 166.3)
- added C25: 47n, Capacitors_SMD:C_0805_HandSoldering, F.Cu at (259.4, 183.9)
- added C26: 47n, Capacitors_SMD:C_0805_HandSoldering, F.Cu at (214.4, 170.5)
- added C27: 470n, Capacitors_SMD:C_0805_HandSoldering, F.Cu at (259.8, 179.8)
- added C28: 47n, Capacitors_SMD:C_0805_HandSoldering, F.Cu at (289.8, 179.5)
- added C29: 100n, Capacitors_SMD:C_0805_HandSoldering, F.Cu at (286.8, 171.3)
- added C3: 100nF, Capacitors_SMD:C_0805_HandSoldering, F.Cu at (268.5, 158.5)
- added C30: 3.3n, Capacitors_SMD:C_0805_HandSoldering, F.Cu at (299.3, 171.5)
- added C31: 33n, Capacitors_SMD:C_0805_HandSoldering, F.Cu at (238.3, 194.7)
- added C32: 3.3n, Capacitors_SMD:C_0805_HandSoldering, F.Cu at (279.6, 183.8)
- added C33: 1u, Capacitors_SMD:C_0805_HandSoldering, F.Cu at (268.9, 182.4)
- added C34: 100n, Capacitors_SMD:C_0805_HandSoldering, F.Cu at (273.9, 187.4)
- added C4: 100nF, Capacitors_SMD:C_0805_HandSoldering, F.Cu at (268.8, 163.1)
- added C5: 22uF, Capacitors_SMD:C_1206_HandSoldering, F.Cu at (257.0, 158.4)
- added C6: 22uF, Capacitors_SMD:C_1206_HandSoldering, F.Cu at (257.2, 163.0)
- added C7: 75pF, Capacitors_SMD:C_0805_HandSoldering, F.Cu at (238.2, 153.3)
- added C8: 470uF, Capacitors_SMD:CP_Elec_10x10.5, F.Cu at (245.1, 110.2)
- added C9: 47uF, low ESR, Capacitors_SMD:CP_Elec_5x5.3, F.Cu at (216.0, 160.4)
- added D1: 1N5819, Diodes_SMD:D_SOD-123, F.Cu at (257.4, 132.4)
- added D10: 1N5819, Diodes_SMD:D_SOD-123, F.Cu at (214.8, 200.3)
- added D11: ESD5Z3.3T1G, Diodes_SMD:D_SOD-523, F.Cu at (205.0, 204.9)
- added D12: ESD5Z3.3T1G, Diodes_SMD:D_SOD-523, F.Cu at (233.3, 212.9)
- added D13: ESD5Z3.3T1G, Diodes_SMD:D_SOD-523, F.Cu at (290.1, 208.0)
- added D14: ESD5Z3.3T1G, Diodes_SMD:D_SOD-523, F.Cu at (220.5, 215.0)
- added D15, D16, D17: ESD5Z3.3T1G, Diodes_SMD:D_SOD-523, F.Cu at (232.5, 160.1)
- added D18: ESD5Z3.3T1G, Diodes_SMD:D_SOD-523, F.Cu at (250.7, 217.2)
- added D2: 1N5819, Diodes_SMD:D_SOD-123, F.Cu at (265.6, 190.8)
- added D3: DB2X41500L, Diodes_SMD:D_SOD-123, F.Cu at (215.5, 122.5)
- added D4: KPT-1608SGC, LEDs:LED_0805_HandSoldering, F.Cu at (252.4, 194.2)
- added D5: 1N5819, Diodes_SMD:D_SOD-123, F.Cu at (264.9, 199.4)
- added D6: 1N5819, Diodes_SMD:D_SOD-123, F.Cu at (276.7, 196.9)
- added D7: KPT-1608SGC, LEDs:LED_0805_HandSoldering, F.Cu at (235.5, 205.1)
- added D8: 1N5819, Diodes_SMD:D_SOD-123, F.Cu at (249.4, 202.3)
- added D9: KPT-1608SGC, LEDs:LED_0805_HandSoldering, F.Cu at (229.0, 205.5)
- added J1: CONN_01X02, Pin_Headers:Pin_Header_Straight_1x02_Pitch1.27mm, F.Cu at (189.7, 211.8)
- added J2: 40HAT, Socket_Strips:Socket_Strip_Straight_2x20_Pitch2.54mm, B.Cu at (208.4, 98.8)
- added J4: Conn_01x06, Mylib:bornier6_2.54, F.Cu at (262.1, 127.0)
- added J5: PWM, Connect:bornier2, F.Cu at (204.2, 133.4)
- added L1: MSS7341-103MLD, Choke_SMD:Choke_SMD_7.3x7.3_H4.5, F.Cu at (204.8, 160.2)
- added MK1: M2.5, Mounting_Holes:MountingHole_2-5mm, F.Cu at (203.5, 97.5)
- added MK2: M2.5, Mounting_Holes:MountingHole_2-5mm, F.Cu at (261.5, 97.5)
- added MK3: M2.5, Mounting_Holes:MountingHole_2-5mm, F.Cu at (203.5, 146.5)
- added MK4: M2.5, Mounting_Holes:MountingHole_2-5mm, F.Cu at (261.5, 146.5)
- added P1: Power jack, Connect:BARREL_JACK, F.Cu at (213.9, 106.4)
- added P10: CONN_01X03, Connect:Fan_Pin_Header_Straight_1x03, F.Cu at (229.8, 169.9)
- added P11: CONN_01X03, Connect:Fan_Pin_Header_Straight_1x03, F.Cu at (222.1, 170.2)
- added P2: Power, Connect:bornier2, F.Cu at (209.0, 116.2)
- added P3: SSR 1, Connect:bornier2, F.Cu at (209.3, 145.9)
- added P4: SSR 2, Connect:bornier2, F.Cu at (219.7, 145.9)
- added P5: SSR 3, Connect:bornier2, F.Cu at (230.1, 145.9)
- added P6: i2c_ext, Connect:Fan_Pin_Header_Straight_1x04, F.Cu at (262.3, 139.8)
- added P7: Ext, Connect:PINHEAD1-6, F.Cu at (260.8, 116.8)
- added P8: CONN_01X03, Connect:Fan_Pin_Header_Straight_1x03, F.Cu at (243.7, 169.8)
- added P9: CONN_01X03, Connect:Fan_Pin_Header_Straight_1x03, F.Cu at (236.9, 170.0)
- added Q3: TSM2306, TO_SOT_Packages_SMD:SOT-23_Handsoldering, F.Cu at (243.7, 156.9)
- added Q4: NTR4503NT1G, TO_SOT_Packages_SMD:SOT-23_Handsoldering, F.Cu at (242.2, 165.1)
- added Q5: NTR4503NT1G, TO_SOT_Packages_SMD:SOT-23_Handsoldering, F.Cu at (251.1, 165.6)
- added Q6: BC817, TO_SOT_Packages_SMD:SOT-23_Handsoldering, F.Cu at (192.9, 168.2)
- added Q7: NTR4503NT1G, TO_SOT_Packages_SMD:SOT-23_Handsoldering, F.Cu at (259.5, 153.0)
- added R1: DNP, Resistors_SMD:R_0805_HandSoldering, F.Cu at (250.3, 184.8)
- added R10: 1k, Resistors_SMD:R_0805_HandSoldering, F.Cu at (277.8, 224.4)
- added R12: 47, Resistors_SMD:R_0805_HandSoldering, F.Cu at (303.7, 210.4)
- added R13: 820, Resistors_SMD:R_0805_HandSoldering, F.Cu at (304.6, 201.2)
- added R14: 511k, Resistors_SMD:R_0805_HandSoldering, F.Cu at (315.3, 216.0)
- added R15: 105k, Resistors_SMD:R_0805_HandSoldering, F.Cu at (310.1, 206.0)
- added R16: 1k, Resistors_SMD:R_0805_HandSoldering, F.Cu at (294.9, 201.9)
- added R17: 820, Resistors_SMD:R_0805_HandSoldering, F.Cu at (320.0, 207.7)
- added R18: 670, Resistors_SMD:R_0805_HandSoldering, F.Cu at (270.3, 225.1)
- added R19: 1k, Resistors_SMD:R_0805_HandSoldering, F.Cu at (328.1, 231.0)
- added R2: 10K, Resistors_SMD:R_0603_HandSoldering, F.Cu at (272.3, 207.8)
- added R20: 1k, Resistors_SMD:R_0805_HandSoldering, F.Cu at (298.6, 227.5)
- added R21: 820, Resistors_SMD:R_0805_HandSoldering, F.Cu at (331.7, 210.6)
- added R22: 49.9, Resistors_SMD:R_0805_HandSoldering, F.Cu at (259.9, 225.2)
- added R25: 10k, Resistors_SMD:R_0805_HandSoldering, F.Cu at (317.3, 198.9)
- added R26: 4,7k, Resistors_SMD:R_0805_HandSoldering, F.Cu at (320.8, 191.0)
- added R27: 4,7k, Resistors_SMD:R_0805_HandSoldering, F.Cu at (311.7, 187.0)
- added R28: 47, Resistors_SMD:R_0805_HandSoldering, F.Cu at (288.2, 202.2)
- added R3: 3.9K, Resistors_SMD:R_0603_HandSoldering, F.Cu at (238.1, 219.5)
- added R30: 10k, Resistors_SMD:R_0805_HandSoldering, F.Cu at (328.6, 221.1)
- added R31: 10k, Resistors_SMD:R_0805_HandSoldering, F.Cu at (304.7, 192.8)
- added R32: 10k, Resistors_SMD:R_0805_HandSoldering, F.Cu at (322.4, 182.4)
- added R33: 470, Resistors_SMD:R_0805_HandSoldering, F.Cu at (327.0, 198.3)
- added R34: 470, Resistors_SMD:R_0805_HandSoldering, F.Cu at (312.4, 197.1)
- added R35: 470, Resistors_SMD:R_0805_HandSoldering, F.Cu at (302.4, 187.4)
- added R36: 470, Resistors_SMD:R_0805_HandSoldering, F.Cu at (297.6, 194.2)
- added R37: 10k, Resistors_SMD:R_0805_HandSoldering, F.Cu at (291.5, 196.4)
- added R38: 820, Resistors_SMD:R_0805_HandSoldering, F.Cu at (310.3, 233.8)
- added R39: 10k, Resistors_SMD:R_0603_HandSoldering, F.Cu at (232.5, 160.1)
- added R4: 3.9K, Resistors_SMD:R_0603_HandSoldering, F.Cu at (223.5, 220.3)
- added R40: 47, Resistors_SMD:R_0603_HandSoldering, F.Cu at (300.5, 237.3)
- added R41, R42, R43, R44, R45, R46: 47, Resistors_SMD:R_0603_HandSoldering, F.Cu at (232.5, 160.1)
- added R5: 10k, Resistors_SMD:R_0603_HandSoldering, F.Cu at (282.1, 218.2)
- added RV1: 1k, Potentiometers:Potentiometer_Trimmer_Bourns_3266W, F.Cu at (252.0, 121.3)
- added SP1: SPEAKER, Capacitors_ThroughHole:CP_Radial_D16.0mm_P7.50mm, F.Cu at (213.6, 133.7)
- added U1: CAT24C32, Housings_SOIC:SOIC-8_3.9x4.9mm_Pitch1.27mm, F.Cu at (242.8, 103.0)
- added U3: LM3940_SOT223, TO_SOT_Packages_SMD:SOT-223-3Lead_TabPin2, F.Cu at (206.2, 172.3)
- added U4: LM321, TO_SOT_Packages_SMD:TSOT-23-5_HandSoldering, F.Cu at (195.0, 153.8)
- added U5: ADS1248, Housings_SSOP:TSSOP-28_4.4x9.7mm_Pitch0.65mm, F.Cu at (236.9, 129.0)
- J3: value 40HAT -> CONN_02X02; footprint Socket_Strips:Socket_Strip_Straight_2x20 -> Pin_Headers:Pin_Header_Straight_2x02_Pitch1.27mm; moved to F.Cu
- Q1: value DMG2305UX -> DMMT5401; footprint TO_SOT_Packages_SMD:SOT-23 -> TO_SOT_Packages_SMD:SOT-23-6_Handsoldering
- Q2: value DMMT5401 -> DMG2305UX; footprint TO_SOT_Packages_SMD:SOT-23-6 -> TO_SOT_Packages_SMD:SOT-23_Handsoldering
- R11: value DNP -> 4.7k
- R23: value 22 -> 100k; footprint Resistors_SMD:R_0603_HandSoldering -> Resistors_SMD:R_0805_HandSoldering
- R24: value 22 -> 13.3k; footprint Resistors_SMD:R_0603_HandSoldering -> Resistors_SMD:R_0805_HandSoldering
- R29: value 10K -> 47; footprint Resistors_SMD:R_0603_HandSoldering -> Resistors_SMD:R_0805_HandSoldering
- R6: value 3.9K -> DNP; footprint Resistors_SMD:R_0603_HandSoldering -> Resistors_SMD:R_0805_HandSoldering
- R8: value 3.9K -> 10k
- R9: value DNP -> 100k
- U2: value CAT24C32 -> TPS54302; footprint Housings_SOIC:SOIC-8_3.9x4.9mm_Pitch1.27mm -> TO_SOT_Packages_SMD:SOT-23-6_Handsoldering
- moved R23 268.3 mm to (311.4, 223.5), turned to 0 degrees
- moved R24 256.5 mm to (302.1, 219.6), turned to 0 degrees
- moved R9 249.2 mm to (293.0, 216.6)
- moved R8 232.7 mm to (286.5, 224.7)
- moved R29 220.3 mm to (306.8, 178.8)
- moved H1 219.5 mm to (272.0, 174.3)
- moved R7 215.1 mm to (261.9, 209.3)
- moved R11 208.0 mm to (271.8, 216.3)
- moved J3 196.4 mm to (242.8, 185.0)
- moved Q2 182.7 mm to (248.4, 160.6)
- moved R6 172.8 mm to (218.3, 207.8)
- moved H2 142.1 mm to (191.8, 196.7)
- moved H3 129.3 mm to (179.7, 198.1)
- moved Q1 127.3 mm to (177.9, 159.3), turned to 0 degrees
- moved U2 125.7 mm to (236.3, 118.0), turned to 0 degrees
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Connections:
- J3 pad 1: /P3V3_HAT -> +3V3
- J3 pad 2: /P5V_HAT -> /P3V3_HAT
- J3 pad 3: (no net) -> P5V
- Q1 pad 2: /P5V_HAT -> Net-(Q1-Pad1)
- Q1 pad 3: /P5V -> Net-(Q1-Pad1)
- Q2 pad 1: Net-(Q2-Pad1) -> Net-(Q1-Pad4)
- Q2 pad 2: Net-(Q2-Pad1) -> /P5V_HAT
- Q2 pad 3: Net-(Q2-Pad1) -> P5V
- R11 pad 1: Net-(J9-Pad2) -> 1Wire
- R11 pad 2: GND -> +3V3
- R23 pad 1: Net-(Q2-Pad1) -> Net-(C7-Pad1)
- R23 pad 2: GND -> Net-(C7-Pad2)
- R24 pad 1: Net-(Q1-Pad1) -> Net-(C7-Pad2)
- R29 pad 1: /P3V3 -> Net-(P6-Pad4)
- R29 pad 2: Net-(J9-Pad2) -> SDA
- R6 pad 1: /P3V3 -> /P3V3_HAT
- R6 pad 2: /ID_SD_EEPROM -> +3V3
- R7 pad 1: /P3V3_HAT -> /P5V_HAT
- R7 pad 2: /P3V3 -> P5V
- R8 pad 1: /P3V3 -> Net-(Q1-Pad4)
- R8 pad 2: /ID_SC_EEPROM -> GND
- R9 pad 1: /P5V_HAT -> GND
- R9 pad 2: /P5V -> PWM2
- U2 pad 2: GND -> Net-(C4-Pad2)
- U2 pad 3: GND -> +VDC
- U2 pad 4: GND -> Net-(C7-Pad2)
- U2 pad 5: /ID_SC_EEPROM -> Net-(R14-Pad2)
- U2 pad 6: /ID_SD_EEPROM -> Net-(C4-Pad1)
Routing:
- net /P3V3: track 31.3 -> 0.00 mm
- net Net-(J9-Pad2): track 9.58 -> 0.00 mm
- net /P5V: track 9.02 -> 0.00 mm
- net /ID_SD_EEPROM: track 8.99 -> 0.00 mm
- net /ID_SC_EEPROM: track 8.17 -> 0.00 mm
- net Net-(Q1-Pad1): track 6.02 -> 0.00 mm
- net /P5V_HAT: track 3.77 -> 0.00 mm
- net Net-(Q2-Pad1): track 3.37 -> 0.00 mm
- net /P3V3_HAT: track 2.88 -> 0.00 mm
- removed copper zone on B.Cu, net /P3V3_HAT
- removed copper zone on F.Cu, net /P5V
- removed copper zone on B.Cu, net /P5V_HAT
- removed copper zone on F.Cu, net /P5V_HAT
- removed copper zone on F.Cu, net GND
- removed copper zone on In2.Cu, net GND
Other:
- outline, holes or cut-outs redrawn
- copper layers 4 -> 2
- net class Default: trace_width 0.15 -> 0.2; via_dia 0.4 -> 0.9; via_drill 0.2 -> 0.6
- net class Power added: clearance 0.2, trace_width 0.5, via_dia 1, via_drill 0.7
- rule pad_to_mask_clearance: 0.2 -> 0
- rule trace_min: 0.15 -> 0.1524
- rule via_min_drill: 0.2 -> 0.5
- rule via_min_size: 0.4 -> 0.8
- board text added: "CAMERA"
- board text added: "DISPLAY"
- board text added: "RASPBERRY-PI 40-PIN ADDON BOARD VIEW FROM TOP NOTE: P1 SHOULD BE FITTED ON THE REVERSE OF THE BOARD ADD EDGE CUTS FROM CAMERA AND DISPLAY PORTS AS REQUIRED"
- board text added: "RJ45"
- board text added: "USB"
- board text removed: "If you want to use an SMT 40-pin header, please move the top edge up by 0.5mm and locate the header in the same location as the current TH part."
- board text removed: "This is a HAT compatible PCB starting design based on the official Raspberry Pi specs at: https://github.com/raspberrypi/hats/blob/master/designguide.md Currently the camera slot and display cutout are not here. See the schematic for the details on the EEPROM and power setup. This board does have the correct components for powering the Pi via the HAT. If you need the Pi to provide 5V or 3.3V, ple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"

Commit message: Continued simplifiying
Parts:
- removed C1, C8: 470uF, Capacitors_SMD:CP_Elec_10x10.5
- removed C10, C12, C13, C14, C33: 1u, Capacitors_SMD:C_0805_HandSoldering
- removed C11: 470uF, low ESR, Capacitors_SMD:CP_Elec_6.3x7.7
- removed C15, C16, C17, C18, C19, C20, C21, C22: 1n, Capacitors_SMD:C_0805_HandSoldering
- removed C2: 10uF, Capacitors_SMD:C_1206_HandSoldering
- removed C23, C25, C26, C28: 47n, Capacitors_SMD:C_0805_HandSoldering
- removed C24, C27: 470n, Capacitors_SMD:C_0805_HandSoldering
- removed C29, C34: 100n, Capacitors_SMD:C_0805_HandSoldering
- removed C3, C4: 100nF, Capacitors_SMD:C_0805_HandSoldering
- removed C30, C32: 3.3n, Capacitors_SMD:C_0805_HandSoldering
- removed C31: 33n, Capacitors_SMD:C_0805_HandSoldering
- removed C5, C6: 22uF, Capacitors_SMD:C_1206_HandSoldering
- removed C7: 75pF, Capacitors_SMD:C_0805_HandSoldering
- removed C9: 47uF, low ESR, Capacitors_SMD:CP_Elec_5x5.3
- removed D1, D10, D2, D5, D6, D8: 1N5819, Diodes_SMD:D_SOD-123
- removed D11, D12, D13, D14, D15, D16, D17, D18: ESD5Z3.3T1G, Diodes_SMD:D_SOD-523
- removed D3: DB2X41500L, Diodes_SMD:D_SOD-123
- removed D4, D7, D9: KPT-1608SGC, LEDs:LED_0805_HandSoldering
- removed H1, H2, H3, H4: 3mm_Mounting_Hole, project_footprints:NPTH_3mm_ID
- removed J1: CONN_01X02, Pin_Headers:Pin_Header_Straight_1x02_Pitch1.27mm
- removed J2: 40HAT, Socket_Strips:Socket_Strip_Straight_2x20_Pitch2.54mm
- removed J3: CONN_02X02, Pin_Headers:Pin_Header_Straight_2x02_Pitch1.27mm
- removed J4: Conn_01x06, Mylib:bornier6_2.54
- removed J5: PWM, Connect:bornier2
- removed L1: MSS7341-103MLD, Choke_SMD:Choke_SMD_7.3x7.3_H4.5
- removed MK1, MK2, MK3, MK4: M2.5, Mounting_Holes:MountingHole_2-5mm
- removed P1: Power jack, Connect:BARREL_JACK
- removed P10, P11, P8, P9: CONN_01X03, Connect:Fan_Pin_Header_Straight_1x03
- removed P2: Power, Connect:bornier2
- removed P3: SSR 1, Connect:bornier2
- removed P4: SSR 2, Connect:bornier2
- removed P5: SSR 3, Connect:bornier2
- removed P6: i2c_ext, Connect:Fan_Pin_Header_Straight_1x04
- removed P7: Ext, Connect:PINHEAD1-6
- removed Q1: DMMT5401, TO_SOT_Packages_SMD:SOT-23-6_Handsoldering
- removed Q2: DMG2305UX, TO_SOT_Packages_SMD:SOT-23_Handsoldering
- removed Q3: TSM2306, TO_SOT_Packages_SMD:SOT-23_Handsoldering
- removed Q4, Q5, Q7: NTR4503NT1G, TO_SOT_Packages_SMD:SOT-23_Handsoldering
- removed Q6: BC817, TO_SOT_Packages_SMD:SOT-23_Handsoldering
- removed R1, R6, R7: DNP, Resistors_SMD:R_0805_HandSoldering
- removed R10, R16, R19, R20: 1k, Resistors_SMD:R_0805_HandSoldering
- removed R11: 4.7k, Resistors_SMD:R_0805_HandSoldering
- removed R12, R28, R29: 47, Resistors_SMD:R_0805_HandSoldering
- removed R13, R17, R21, R38: 820, Resistors_SMD:R_0805_HandSoldering
- removed R14: 511k, Resistors_SMD:R_0805_HandSoldering
- removed R15: 105k, Resistors_SMD:R_0805_HandSoldering
- removed R18: 670, Resistors_SMD:R_0805_HandSoldering
- removed R2: 10K, Resistors_SMD:R_0603_HandSoldering
- removed R22: 49.9, Resistors_SMD:R_0805_HandSoldering
- removed R23, R9: 100k, Resistors_SMD:R_0805_HandSoldering
- removed R24: 13.3k, Resistors_SMD:R_0805_HandSoldering
- removed R25, R30, R31, R32, R37: 10k, Resistors_SMD:R_0805_HandSoldering
- removed R26, R27: 4,7k, Resistors_SMD:R_0805_HandSoldering
- removed R3, R4: 3.9K, Resistors_SMD:R_0603_HandSoldering
- removed R33, R34, R35, R36: 470, Resistors_SMD:R_0805_HandSoldering
- removed R39, R5, R8: 10k, Resistors_SMD:R_0603_HandSoldering
- removed R40, R41, R42, R43, R44, R45, R46: 47, Resistors_SMD:R_0603_HandSoldering
- removed RV1: 1k, Potentiometers:Potentiometer_Trimmer_Bourns_3266W
- removed SP1: SPEAKER, Capacitors_ThroughHole:CP_Radial_D16.0mm_P7.50mm
- removed U1: CAT24C32, Housings_SOIC:SOIC-8_3.9x4.9mm_Pitch1.27mm
- removed U2: TPS54302, TO_SOT_Packages_SMD:SOT-23-6_Handsoldering
- removed U3: LM3940_SOT223, TO_SOT_Packages_SMD:SOT-223-3Lead_TabPin2
- removed U4: LM321, TO_SOT_Packages_SMD:TSOT-23-5_HandSoldering
- removed U5: ADS1248, Housings_SSOP:TSSOP-28_4.4x9.7mm_Pitch0.65mm
- added C201: 470uF, Capacitors_SMD:CP_Elec_10x10.5, F.Cu at (232.5, 160.1)
- added C202: 47uF, low ESR, Capacitors_SMD:CP_Elec_5x5.3, F.Cu at (232.5, 160.1)
- added C203, C205, C206, C207, C309: 1u, Capacitors_SMD:C_0805_HandSoldering, F.Cu at (232.5, 160.1)
- added C204: 470uF, low ESR, Capacitors_SMD:CP_Elec_6.3x7.7, F.Cu at (232.5, 160.1)
- added C301, C302, C303, C304: 1n, Capacitors_SMD:C_0805_HandSoldering, F.Cu at (232.5, 160.1)
- added C305, C310: 100n, Capacitors_SMD:C_0805_HandSoldering, F.Cu at (232.5, 160.1)
- added C306, C308: 3.3n, Capacitors_SMD:C_0805_HandSoldering, F.Cu at (232.5, 160.1)
- added C307: 33n, Capacitors_SMD:C_0805_HandSoldering, F.Cu at (232.5, 160.1)
- added D201, D202, D205, D206, D208, D210: 1N5819, Diodes_SMD:D_SOD-123, F.Cu at (232.5, 160.1)
- added D203: DB2X41500L, Diodes_SMD:D_SOD-123, F.Cu at (232.5, 160.1)
- added D204, D207, D209: KPT-1608SGC, LEDs:LED_0805_HandSoldering, F.Cu at (232.5, 160.1)
- added D301, D302, D303, D304: ESD5Z3.3T1G, Diodes_SMD:D_SOD-523, F.Cu at (232.5, 160.1)
- added H101, H102, H103, H104: 3mm_Mounting_Hole, project_footprints:NPTH_3mm_ID, F.Cu at (232.5, 160.1)
- added J101: CONN_01X02, Pin_Headers:Pin_Header_Straight_1x02_Pitch1.27mm, F.Cu at (232.5, 160.1)
- added J102: 40HAT, Pin_Headers:Pin_Header_Straight_2x20_Pitch2.54mm, F.Cu at (206.1, 100.2)
- added J103: CONN_02X02, Pin_Headers:Pin_Header_Straight_2x02_Pitch1.27mm, F.Cu at (232.5, 160.1)
- added J201: Conn_01x06, project_footprints:bornier6_2.54, F.Cu at (232.5, 160.1)
- added J202: PWM, Connectors_Terminal_Blocks:TerminalBlock_bornier-2_P5.08mm, F.Cu at (232.5, 160.1)
- added P201: Power jack, Connectors:BARREL_JACK, F.Cu at (232.5, 160.1)
- added P202: Power, Connectors_Terminal_Blocks:TerminalBlock_bornier-2_P5.08mm, F.Cu at (232.5, 160.1)
- added P203: SSR 1, Connectors_Terminal_Blocks:TerminalBlock_bornier-2_P5.08mm, F.Cu at (232.5, 160.1)
- added P204: SSR 2, Connectors_Terminal_Blocks:TerminalBlock_bornier-2_P5.08mm, F.Cu at (232.5, 160.1)
- added P205: SSR 3, Connectors_Terminal_Blocks:TerminalBlock_bornier-2_P5.08mm, F.Cu at (232.5, 160.1)
- added P206: i2c_ext, Connectors:Fan_Pin_Header_Straight_1x04, F.Cu at (232.5, 160.1)
- added P207: Ext, Connectors:PINHEAD1-6, F.Cu at (232.5, 160.1)
- added P301, P302, P303, P304: CONN_01X03, Connectors:Fan_Pin_Header_Straight_1x03, F.Cu at (232.5, 160.1)
- added Q101: DMMT5401, TO_SOT_Packages_SMD:SOT-23-6_Handsoldering, F.Cu at (232.5, 160.1)
- added Q102: DMG2305UX, TO_SOT_Packages_SMD:SOT-23_Handsoldering, F.Cu at (232.5, 160.1)
- added Q201: TSM2306, TO_SOT_Packages_SMD:SOT-23_Handsoldering, F.Cu at (232.5, 160.1)
- added Q202, Q203, Q205: NTR4503NT1G, TO_SOT_Packages_SMD:SOT-23_Handsoldering, F.Cu at (232.5, 160.1)
- added Q204: BC817, TO_SOT_Packages_SMD:SOT-23_Handsoldering, F.Cu at (232.5, 160.1)
- added R101, R106, R107: DNP, Resistors_SMD:R_0805_HandSoldering, F.Cu at (232.5, 160.1)
- added R102: 10K, Resistors_SMD:R_0603_HandSoldering, F.Cu at (232.5, 160.1)
- added R103, R104: 3.9K, Resistors_SMD:R_0603_HandSoldering, F.Cu at (232.5, 160.1)
- added R105, R108, R303: 10k, Resistors_SMD:R_0603_HandSoldering, F.Cu at (232.5, 160.1)
- added R201: 100k, Resistors_SMD:R_0805_HandSoldering, F.Cu at (232.5, 160.1)
- added R202, R206, R209, R210: 1k, Resistors_SMD:R_0805_HandSoldering, F.Cu at (232.5, 160.1)
- added R203: 4.7k, Resistors_SMD:R_0805_HandSoldering, F.Cu at (232.5, 160.1)
- added R204, R215, R216: 47, Resistors_SMD:R_0805_HandSoldering, F.Cu at (232.5, 160.1)
- added R205, R207, R211, R302: 820, Resistors_SMD:R_0805_HandSoldering, F.Cu at (232.5, 160.1)
- added R208: 670, Resistors_SMD:R_0805_HandSoldering, F.Cu at (232.5, 160.1)
- added R212, R217, R218, R219, R301: 10k, Resistors_SMD:R_0805_HandSoldering, F.Cu at (232.5, 160.1)
- added R213, R214: 4,7k, Resistors_SMD:R_0805_HandSoldering, F.Cu at (232.5, 160.1)
- added R304, R305, R306, R307, R308, R309, R310: 47, Resistors_SMD:R_0603_HandSoldering, F.Cu at (232.5, 160.1)
- added RV201: 1k, Potentiometers:Potentiometer_Trimmer_Bourns_3266W, F.Cu at (232.5, 160.1)
- added SP201: SPEAKER, Capacitors_THT:CP_Radial_D12.5mm_P7.50mm, F.Cu at (232.5, 160.1)
- added U101: CAT24C32, Housings_SOIC:SOIC-8_3.9x4.9mm_Pitch1.27mm, F.Cu at (232.5, 160.1)
- added U201: BuckModule, project_footprints:Buck-Module-1, F.Cu at (213.2, 121.6)
- added U202: LM3940_SOT223, TO_SOT_Packages_SMD:SOT-223-3_TabPin2, F.Cu at (232.5, 160.1)
- added U203: LM321, TO_SOT_Packages_SMD:TSOT-23-5_HandSoldering, F.Cu at (232.5, 160.1)
- added U301: ADS1248, Housings_SSOP:TSSOP-28_4.4x9.7mm_Pitch0.65mm, F.Cu at (232.5, 160.1)
Other:
- net class Default: trace_width 0.2 -> 0.25
- net class Power: trace_width 0.5 -> 0.8
- net class power2 added: clearance 0.15, trace_width 0.75, via_dia 0.8, via_drill 0.6
