File: Arpette.sch (KiCad schematic (older format))
At the start: 18 parts, among them J1 CONN_01X02, J2 40HAT, J3 CONN_02X02, Q1 DMMT5401, Q2 DMG2305UX, U1 CAT24C32

Commit message: Continued simplifiying
Parts:
- renumbered H1 to H101, H2 to H102, H3 to H103, H4 to H104, J1 to J101, J2 to J102, J3 to J103, Q1 to Q101, Q2 to Q102, R1 to R101, R2 to R102, R3 to R103, R4 to R104, R5 to R105, R6 to R106, R7 to R107, R8 to R108, U1 to U101
Changed lines of the file:
@@
 LIBS:valves
 LIBS:raspberrypi_hat
+LIBS:Arpette
 LIBS:Arpette-cache
 EELAYER 25 0
@@
 $EndDescr
 $Comp
-L 3mm_Mounting_Hole H1
+L 3mm_Mounting_Hole H101
 U 1 1 5834BC4A
 P 5650 6000
-F 0 "H1" H 5500 6100 60  0000 C CNN
+F 0 "H101" H 5500 6100 60  0000 C CNN
 F 1 "3mm_Mounting_Hole" H 5650 5850 60  0000 C CNN
 F 2 "project_footprints:NPTH_3mm_ID" H 5550 6000 60  0001 C CNN
@@
 $EndComp
 $Comp
-L 3mm_Mounting_Hole H3
+L 3mm_Mounting_Hole H103
 U 1 1 5834BCDF
 P 6650 6000
-F 0 "H3" H 6500 6100 60  0000 C CNN
+F 0 "H103" H 6500 6100 60  0000 C CNN
 F 1 "3mm_Mounting_Hole" H 6650 5850 60  0000 C CNN
 F 2 "project_footprints:NPTH_3mm_ID" H 6550 6000 60  0001 C CNN
@@
 $EndComp
 $Comp
-L 3mm_Mounting_Hole H2
+L 3mm_Mounting_Hole H102
 U 1 1 5834BD62
 P 5650 6550
-F 0 "H2" H 5500 6650 60  0000 C CNN
+F 0 "H102" H 5500 6650 60  0000 C CNN
 F 1 "3mm_Mounting_Hole" H 5650 6400 60  0000 C CNN
 F 2 "project_footprints:NPTH_3mm_ID" H 5550 6550 60  0001 C CNN
@@
 $EndComp
 $Comp
-L 3mm_Mounting_Hole H4
+L 3mm_Mounting_Hole H104
 U 1 1 5834BDED
 P 6700 6550
-F 0 "H4" H 6550 6650 60  0000 C CNN
+F 0 "H104" H 6550 6650 60  0000 C CNN
 F 1 "3mm_Mounting_Hole" H 6700 6400 60  0000 C CNN
 F 2 "project_footprints:NPTH_3mm_ID" H 6600 6550 60  0001 C CNN
@@
 $EndComp
 $Comp
-L OX40HAT J2
+L OX40HAT J102
 U 1 1 58DFC771
 P 2600 2250
-F 0 "J2" H 2950 2350 50  0000 C CNN
+F 0 "J102" H 2950 2350 50  0000 C CNN
 F 1 "40HAT" H 2300 2350 50  0000 C CNN
 F 2 "Pin_Headers:Pin_Header_Straight_2x20_Pitch2.54mm" H 2600 2450 50  0000 C CNN
@@
 P3V3
 $Comp
-L CONN_02X02 J3
+L CONN_02X02 J103
 U 1 1 58E13683
 P 6100 4650
-F 0 "J3" H 6100 4800 50  0000 C CNN
+F 0 "J103" H 6100 4800 50  0000 C CNN
 F 1 "CONN_02X02" H 6100 4500 50  0000 C CNN
 F 2 "Pin_Headers:Pin_Header_Straight_2x02_Pitch1.27mm" H 6100 3450 50  0001 C CNN
@@
 This is the recommended 5V rail protection for \na HAT with power going to the Pi.\nSee https://github.com/raspberrypi/hats/blob/master/designguide.md#back-powering-the-pi-via-the-j8-gpio-header
 $Comp
-L DMG2305UX Q2
+L DMG2305UX Q102
 U 1 1 58E14EB1
 P 6150 2400
-F 0 "Q2" V 6300 2550 50  0000 R CNN
+F 0 "Q102" V 6300 2550 50  0000 R CNN
 F 1 "DMG2305UX" V 6300 2350 50  0000 R CNN
 F 2 "TO_SOT_Packages_SMD:SOT-23_Handsoldering" H 6350 2500 50  0001 C CNN
@@
 $EndComp
 $Comp
-L DMMT5401 Q1
+L DMMT5401 Q101
 U 1 1 58E1538B
 P 5850 3000
-F 0 "Q1" H 6050 3075 50  0000 L CNN
+F 0 "Q101" H 6050 3075 50  0000 L CNN
 F 1 "DMMT5401" H 6050 3000 50  0000 L CNN
 F 2 "TO_SOT_Packages_SMD:SOT-23-6_Handsoldering" H 6050 2925 50  0000 L CIN
@@
 $EndComp
 $Comp
-L DMMT5401 Q1
+L DMMT5401 Q101
 U 2 1 58E153D6
 P 6450 3000
-F 0 "Q1" H 6650 3075 50  0000 L CNN
+F 0 "Q101" H 6650 3075 50  0000 L CNN
 F 1 "DMMT5401" H 6650 3000 50  0000 L CNN
 F 2 "TO_SOT_Packages_SMD:SOT-23-6_Handsoldering" H 6650 2925 50  0000 L CIN
@@
 $EndComp
 $Comp
-L R R5
+L R R105
 U 1 1 58E15896
 P 5750 3600
-F 0 "R5" V 5830 3600 50  0000 C CNN
+F 0 "R105" V 5830 3600 50  0000 C CNN
 F 1 "10k" V 5750 3600 50  0000 C CNN
 F 2 "Resistors_SMD:R_0603_HandSoldering" V 5680 3600 50  0001 C CNN
@@
 $EndComp
 $Comp
-L R R8
+L R R108
 U 1 1 58E158A1
 P 6550 3600
-F 0 "R8" V 6630 3600 50  0000 C CNN
+F 0 "R108" V 6630 3600 50  0000 C CNN
 F 1 "10k" V 6550 3600 50  0000 C CNN
 F 2 "Resistors_SMD:R_0603_HandSoldering" V 6480 3600 50  0001 C CNN
@@
 Connection ~ 6550 2400
 $Comp
-L CAT24C32 U1
+L CAT24C32 U101
 U 1 1 58E1713F
 P 2100 5850
-F 0 "U1" H 2450 6200 50  0000 C CNN
+F 0 "U101" H 2450 6200 50  0000 C CNN
 F 1 "CAT24C32" H 1850 6200 50  0000 C CNN
 F 2 "Housings_SOIC:SOIC-8_3.9x4.9mm_Pitch1.27mm" H 2100 5850 50  0001 C CNN
@@
 $EndComp
 $Comp
-L R R3
+L R R103
 U 1 1 58E17715
 P 2350 7400
-F 0 "R3" V 2430 7400 50  0000 C CNN
+F 0 "R103" V 2430 7400 50  0000 C CNN
 F 1 "3.9K" V 2350 7400 50  0000 C CNN
 F 2 "Resistors_SMD:R_0603_HandSoldering" V 2280 7400 50  0001 C CNN
@@
 $EndComp
 $Comp
-L R R4
+L R R104
 U 1 1 58E17720
 P 2350 7650
-F 0 "R4" V 2430 7650 50  0000 C CNN
+F 0 "R104" V 2430 7650 50  0000 C CNN
 F 1 "3.9K" V 2350 7650 50  0000 C CNN
 F 2 "Resistors_SMD:R_0603_HandSoldering" V 2280 7650 50  0001 C CNN
@@
 ID_SC_EEPROM_pu
 $Comp
-L CONN_01X02 J1
+L CONN_01X02 J101
 U 1 1 58E18D32
 P 750 6050
-F 0 "J1" H 750 6200 50  0000 C CNN
+F 0 "J101" H 750 6200 50  0000 C CNN
 F 1 "CONN_01X02" V 850 6050 50  0000 C CNN
 F 2 "Pin_Headers:Pin_Header_Straight_1x02_Pitch1.27mm" H 750 6050 50  0001 C CNN
@@
 $EndComp
 $Comp
-L R R2
+L R R102
 U 1 1 58E19E51
 P 1550 6250
-F 0 "R2" V 1630 6250 50  0000 C CNN
+F 0 "R102" V 1630 6250 50  0000 C CNN
 F 1 "10K" V 1550 6250 50  0000 C CNN
 F 2 "Resistors_SMD:R_0603_HandSoldering" V 1480 6250 50  0001 C CNN
@@
 EEPROM WRITE ENABLE
 $Comp
-L R R6
+L R R106
 U 1 1 58E22085
 P 6100 4300
-F 0 "R6" V 6180 4300 50  0000 C CNN
+F 0 "R106" V 6180 4300 50  0000 C CNN
 F 1 "DNP" V 6100 4300 50  0000 C CNN
 F 2 "Resistors_SMD:R_0805_HandSoldering" V 6030 4300 50  0001 C CNN
@@
 $EndComp
 $Comp
-L R R7
+L R R107
 U 1 1 58E2218F
 P 6100 4950
-F 0 "R7" V 6180 4950 50  0000 C CNN
+F 0 "R107" V 6180 4950 50  0000 C CNN
 F 1 "DNP" V 6100 4950 50  0000 C CNN
 F 2 "Resistors_SMD:R_0805_HandSoldering" V 6030 4950 50  0001 C CNN
@@
 Connection ~ 5750 4600
 $Comp
-L R R1
+L R R101
 U 1 1 58E22900
 P 1300 6100
-F 0 "R1" V 1380 6100 50  0000 C CNN
+F 0 "R101" V 1380 6100 50  0000 C CNN
 F 1 "DNP" V 1300 6100 50  0000 C CNN
 F 2 "Resistors_SMD:R_0805_HandSoldering" V 1230 6100 50  0001 C CNN
